Commit message: URDs fix

File: src/my_robot_bringup/urdf/robo_cayote.urdf (robot description, URDF)
Before this commit: robot robo_cayote, 35 links, 34 joints
Links:
- removed link ultrasonic_side_left_back_link
- removed link ultrasonic_side_left_front_link
- removed link ultrasonic_side_right_back_link
- removed link ultrasonic_side_right_front_link
Joints:
- removed joint base_link_ultrasonic_side_left_back_joint
- removed joint base_link_ultrasonic_side_left_front_joint
- removed joint base_link_ultrasonic_side_right_back_joint
- removed joint base_link_ultrasonic_side_right_front_joint
